File: hardware/ref_design/board/battler.kicad_sch (KiCad schematic)
At the start: 9 parts

Commit message: Reference design: discrete backlight current sinks replace the AP3156
The AP3156 charge pump (U6, C443652) is out of stock at JLC and LCSC. Each
of the panel's two cathode pins now has its own linear current sink: half
of an MCP6002 (U6, C7377 Preferred) drives an AO3400A (Q5/Q6, C20917 Basic)
and holds a 2.2 ohm sense resistor (R52/R53) at BL_REF. LED_A is on VSYS
through JP2. GPIO44 (now BL_PWM, PWM10 A) sets BL_REF through 100k/3.9k
and 1 uF: 0.124 V at 100% = 56 mA a pin, 113 mA in all (panel max 120).
RG 330 ohm, RF 10k, CF 1 nF, gate pull-downs 100k: simulated first
(board/sim, previous commit), phase margin >= 72.5 deg at every corner.

Every new part is Basic or Preferred: 12 extended part numbers instead of
13, parts $4.77 a board instead of $5.01, about $16.81 a unit at 10.

Layout: the sinks sit above J3's LED pins between J3 and J2, clear of the
ground bar route.py lays over J3's grounded pins; board rebuilt and
re-routed (route.py, 80 passes): DRC 0 errors, 0 unconnected, 0 parity,
2 cosmetic warnings as before. check_netlist, check_pins (29 parts, 244
pins, 94 passives), ERC 0, check_fit pass. silk.py puts J2's BATT label
above it (the op-amp is now on its left).

Docs: pin reviews for U6 and Q5/Q6 with page cites, passives, U4 (GPIO44)
and the panel; pinmap (GPIO44 PWM, backlight section), bring-up step 5,
design review, PLAN (also: the USB series resistors are 27 ohm, not 22),
BOM, assembly, validation plan items, SOURCES.

Co-Authored-By: Claude Opus 5.5 <noreply@anthropic.com>
Claude-Session: https://claude.ai/code/session_01Ceq1EsbekLwXHokcQ73Ldk
Other:
- note added: "panel, backlight current sinks"
- note removed: "panel, AP3156 backlight driver"
Changed lines of the file:
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@@
         (size 1 1)))
 )
-  (text "panel, AP3156 backlight driver"
+  (text "panel, backlight current sinks"
     (at 99.06 108.5 0)
     (effects
