File: hardware/ref_design/board/power.kicad_sch (KiCad schematic)
At the start: 19 parts, among them Q1 2N7002, U3 ME6211C33M5G

Commit message: Reference design: checklist changes and the datasheet pin gate
Board: PWR_HOLD pull-down (R42, also covers RP2350-E9), charge current
3.3k (333-364 mA), firmware charge pause (CHG_OFF, Q4), R13 33k, 0.1 ohm
in D5's path, JP1/JP2 cut-jumpers, TP6-8, spare 1206 footprints, 4-bit
revision strap on GPIO22-25 (REV 1 on the back).

Datasheet review of every part's pins (pin_review/, tools/check_pins.py)
found and fixed: J6 TX/RX swapped against Raspberry Pi's debug connector
spec, USB series resistors 22 to 27 ohm, the ME6211 CE able to lead its
VIN at a live plug-in (C47 on PWR_EN).

Case: silicone height 1.2 mm from the DS Lite, chamfered step.

Co-Authored-By: Claude Opus 5.5 <noreply@anthropic.com>
Claude-Session: https://claude.ai/code/session_01MUt6paNsT75sqwAr83zRS3
Parts:
- added C47: 100n, Capacitor_SMD:C_0402_1005Metric, symbol Device:C
- added JP1: Bridged, Jumper:SolderJumper-2_P1.3mm_Bridged_Pad1.0x1.5mm, symbol Jumper:SolderJumper_2_Bridged
- added R42: 4.7k, Resistor_SMD:R_0402_1005Metric, symbol Device:R
- added TP6: PWR_EN, TestPoint:TestPoint_Pad_D1.0mm, symbol Connector:TestPoint
- added TP7: LS_GATE, TestPoint:TestPoint_Pad_D1.0mm, symbol Connector:TestPoint
- added TP8: AMP_SHDN, TestPoint:TestPoint_Pad_D1.0mm, symbol Connector:TestPoint
- R13: value 100k -> 33k; LCSC C25741 -> C25779; MPN 0402WGF1003TCE -> 0402WGF3302TCE
Connections:
- net +3V3: now also JP1.2 (B); no longer C6.1, C7.1, U3.5 (V_{OUT})
- net GND: now also C47.2, R42.2
- net PWR_EN: now also C47.1, TP6.1
- net PWR_HOLD: now also R42.1
- new net 3V3_LDO: C6.1, C7.1, JP1.1 (A), U3.5 (V_{OUT})
- new net AMP_SHDN: TP8.1
- new net LS_GATE: TP7.1
