File: hardware/ref_design/board/storage.kicad_sch (KiCad schematic)
At the start: 10 parts, among them J8 DM3AT-SF-PEJM5

Commit message: ref_design ESP32-S3: first placement (module, microSD slot with trimmed front tabs, series resistors, third register; case grow_l 1.5 for the shell tabs' copper edge), BOOT/RESET buttons dropped (J7 pads stay), place_new.py, antenna keepout, module GND vias; not routed
Co-Authored-By: Claude Sonnet 5.5 <noreply@anthropic.com>
Parts:
- J8: footprint Connector_Card:microSD_HC_Hirose_DM3AT-SF-PEJM5 -> battler:microSD_HC_Hirose_DM3AT-SF-PEJM5
Changed lines of the file:
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@@
 			)
 		)
-		(property "Footprint" "Connector_Card:microSD_HC_Hirose_DM3AT-SF-PEJM5"
+		(property "Footprint" "battler:microSD_HC_Hirose_DM3AT-SF-PEJM5"
 			(at 139.7 96.52 0)
 			(hide yes)
